Commit message: You work, thx. Now please donwload

File: exam-1.7/urdf/exam_robot.urdf (robot description, URDF)
Before this commit: robot exam_robot, 6 links, 5 joints
Links:
- removed link wheel_left_back_link
- removed link wheel_left_front_link
- removed link wheel_right_back_link
- removed link wheel_right_front_link
- added link left_wheel; visual cylinder length=0.04 radius=0.08
- added link right_wheel; visual cylinder length=0.04 radius=0.08
- link base_link: geometry visual box size=0.4 0.3 0.1
- link sensor_link: geometry visual box size=0.05 0.05 0.05
Joints:
- removed joint base_to_left_back_wheel
- removed joint base_to_left_front_wheel
- removed joint base_to_right_back_wheel
- removed joint base_to_right_front_wheel
- added joint base_to_left_wheel: type continuous, parent base_link, child left_wheel, origin xyz=0 0.17 0 rpy=1.5708 0 0, axis 0 0 1
- added joint base_to_right_wheel: type continuous, parent base_link, child right_wheel, origin xyz=0 -0.17 0 rpy=1.5708 0 0, axis 0 0 1
- joint base_to_sensor: origin xyz=0.15 0 0.1 -> xyz=0.2 0 0.08
